File: 100 - Analog Electronics Fundamentals/Analog Electronics Fundamentals 103 - Lab1 Schematic.sch (EAGLE design)
At the start: 7 parts, among them T1 2N2222

Commit message: For Workshop 103, lab1, changed R1 to be 3.2k instead of 10k (10k didn't provide enough current).  Also added AN1707 to Workshop 102
Parts:
- R1: value 10k -> 3.2k
Changed lines of the file:
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@@
 <parts>
 <part name="9V" library="battery" deviceset="AB9V" device=""/>
-<part name="R1" library="resistor" deviceset="R-US_" device="0204/7" value="10k"/>
+<part name="R1" library="resistor" deviceset="R-US_" device="0204/7" value="3.2k"/>
 <part name="R2" library="resistor" deviceset="R-US_" device="0204/7" value="1k"/>
 <part name="GND1" library="supply1" deviceset="GND" device=""/>
